File: schematic/scraptcha.sch (EAGLE design)
At the start: 28 parts, among them J1 1X5, Q2 2N2907, Q3 2N2907, Q4 2N2907, U1 PI_COBBLER, U2 74LS595D, U3 MCP2300X/SO, U4 74LS595N, X1 HD44780LCD-1602

Commit message: Added updated schematic
Parts:
- R10, R8, R9: value 33ohm -> 100ohm
Other:
- note added: "Engineer: Matt Staniszewski"
- note added: "LCD"
- note added: "LEDs"
- note added: "Webcam"
Changed lines of the file:
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@@
 <part name="C2" library="adafruit" deviceset="C-US" device="C0805K" value="0.1uF"/>
 <part name="U1" library="scraptcha" deviceset="PI_COBBLER" device=""/>
-<part name="R8" library="adafruit" deviceset="R-US_" device="0204/5" value="33ohm"/>
-<part name="R9" library="adafruit" deviceset="R-US_" device="0204/5" value="33ohm"/>
-<part name="R10" library="adafruit" deviceset="R-US_" device="0204/5" value="33ohm"/>
+<part name="R8" library="adafruit" deviceset="R-US_" device="0204/5" value="100ohm"/>
+<part name="R9" library="adafruit" deviceset="R-US_" device="0204/5" value="100ohm"/>
+<part name="R10" library="adafruit" deviceset="R-US_" device="0204/5" value="100ohm"/>
 <part name="5V)" library="supply1" deviceset="VCC" device="" value="5V0"/>
-<part name="P+13" library="supply1" deviceset="VCC" device="" value="3V3"/>
-<part name="P+14" library="supply1" deviceset="VCC" device="" value="3V3"/>
-<part name="P+15" library="supply1" deviceset="VCC" device="" value="3V3"/>
+<part name="P+13" library="supply1" deviceset="VCC" device="" value="5V0"/>
+<part name="P+14" library="supply1" deviceset="VCC" device="" value="5V0"/>
+<part name="P+15" library="supply1" deviceset="VCC" device="" value="5V0"/>
 <part name="P+16" library="supply1" deviceset="VCC" device=""/>
 <part name="GND11" library="supply1" deviceset="GND" device=""/>
@@
 <part name="GND12" library="supply1" deviceset="GND" device=""/>
 <part name="GND13" library="supply1" deviceset="GND" device=""/>
+<part name="FRAME1" library="frames" deviceset="LETTER_L" device=""/>
 </parts>
 <sheets>
@@
 <text x="25.4" y="68.58" size="2.54" layer="96" align="center">Logitech C310
 Webcam</text>
+<wire x1="-233.68" y1="109.22" x2="157.48" y2="109.22" width="0.1524" layer="94"/>
+<wire x1="157.48" y1="109.22" x2="157.48" y2="-157.48" width="0.1524" layer="94"/>
+<wire x1="157.48" y1="-157.48" x2="-233.68" y2="-157.48" width="0.1524" layer="94"/>
+<wire x1="-233.68" y1="-157.48" x2="-233.68" y2="109.22" width="0.1524" layer="94"/>
+<text x="58.42" y="-129.54" size="2.54" layer="94">Engineer: Matt Staniszewski</text>
+<text x="-137.16" y="91.44" size="6.4516" layer="94">LCD</text>
+<text x="-88.9" y="-121.92" size="6.4516" layer="94">LEDs</text>
+<text x="7.62" y="86.36" size="6.4516" layer="94">Webcam</text>
 </plain>
 <instances>
@@
 <instance part="GND12" gate="1" x="81.28" y="-71.12"/>
 <instance part="GND13" gate="1" x="127" y="-71.12"/>
+<instance part="FRAME1" gate="G$2" x="55.88" y="-157.48"/>
 </instances>
 <busses>
